File: native/parity/docs-oracle/board/oracle.kicad_pcb (KiCad board)
At the start: 2 copper layers, 240 x 190 mm, 71 parts, among them J1 PinHeader_1x04_P2.54mm_Vertic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, J10 OffsetDrills, J11 OffsetDrills, J12 OffsetDrills, J13 OffsetDrills, J14 OffsetDrills, J15 PinHeader_1x04_P2.54mm_Vertic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, J16 PinHeader_1x04_P2.54mm_Vertic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, J17 PinHeader_1x04_P2.54mm_Vertic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, J18 PinHeader_1x04_P2.54mm_Vertic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, J19 PinHeader_1x04_P2.54mm_Vertic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, J2 PinHeader_1x04_P2.54mm_Vertic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, J20 PinHeader_1x04_P2.54mm_Vertic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, J21 PinHeader_1x04_P2.54mm_Vertic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, J22 OffsetDrills, J23 OffsetDrills, J24 OffsetDrills, J25 OffsetDrills, J26 OffsetDrills, J27 OffsetDrills, J28 OffsetDrills, J3 PinHeader_1x04_P2.54mm_Vertic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, J4 PinHeader_1x04_P2.54mm_Vertic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, J5 PinHeader_1x04_P2.54mm_Vertic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, J6 PinHeader_1x04_P2.54mm_Vertic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, J7 PinHeader_1x04_P2.54mm_Vertic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, J8 OffsetDrills, J9 OffsetDrills, Q1 SOT-23, Q10 SOT-23, Q11 SOT-23, Q12 SOT-23, Q13 SOT-23, Q14 SOT-23, Q2 SOT-23, Q3 SOT-23, Q4 SOT-23, Q5 SOT-23, Q6 SOT-23, Q7 SOT-23, Q8 SOT-23, Q9 SOT-23, U1 SOIC-8_3.9x4.9mm_P1.27mm, U10 SOIC-8_3.9x4.9mm_P1.27mm, U11 SOIC-8_3.9x4.9mm_P1.27mm, U12 SOIC-8_3.9x4.9mm_P1.27mm, U13 SOIC-8_3.9x4.9mm_P1.27mm, U14 SOIC-8_3.9x4.9mm_P1.27mm, U2 SOIC-8_3.9x4.9mm_P1.27mm, U3 SOIC-8_3.9x4.9mm_P1.27mm, U4 SOIC-8_3.9x4.9mm_P1.27mm, U5 SOIC-8_3.9x4.9mm_P1.27mm, U6 SOIC-8_3.9x4.9mm_P1.27mm, U7 SOIC-8_3.9x4.9mm_P1.27mm, U8 SOIC-8_3.9x4.9mm_P1.27mm, U9 SOIC-8_3.9x4.9mm_P1.27mm

Commit message: test(parity): grow the docs oracle with unusual shapes; KiCad's pad outlines
The oracle board is now written as KiCad 10 text (no pcbnew) and finished by
KiCad over its IPC API, which fills the zones, saves the board and dumps every
pad's outline on every copper layer. New: a four-layer stackup, an arc-cornered
outline with a notch and two cutouts, custom pads (polygon, circle and arc
primitives), chamfered, round-rect, trapezoid and odd-angle oval pads,
castellated, press-fit, counterbored and countersunk pads, every via span
including a backdrill, arc tracks, an arc-edged zone and a keep-out.

PcbPad::copper_outline / copper_rings give a pad's copper as KiCad shapes it;
docs_oracle.rs checks drill centres on every span, backdrills, flashes on all
four copper layers and every pad outline against KiCad.

Co-Authored-By: Claude Opus 5.5 <noreply@anthropic.com>
Parts:
- added J90: EdgePads, Oracle:EdgePads, F.Cu at (0.00, 110.0)
- added J91: ArcLink, Oracle:ArcLink, F.Cu at (120.0, 150.0)
- added U100: UnusualPads, Oracle:UnusualPads, F.Cu at (35.0, 175.0)
- added U101: UnusualPads, Oracle:UnusualPads, F.Cu at (90.0, 175.0)
- added U102: UnusualPads, Oracle:UnusualPads, F.Cu at (145.0, 175.0)
- added U103: UnusualPads, Oracle:UnusualPads, F.Cu at (200.0, 175.0)
- added U104: UnusualPads, Oracle:UnusualPads, B.Cu at (35.0, 225.0)
- added U105: UnusualPads, Oracle:UnusualPads, B.Cu at (90.0, 225.0)
- added U106: UnusualPads, Oracle:UnusualPads, B.Cu at (145.0, 225.0)
- added U107: UnusualPads, Oracle:UnusualPads, B.Cu at (200.0, 225.0)
Routing:
- net SIG_LINK: track 0.00 -> 30.0 mm
- net GND: track 0.00 -> 24.2 mm, vias 0 -> 1
- net SIG_B: track 0.00 -> 18.0 mm, vias 0 -> 2
- net SIG_A: track 0.00 -> 18.0 mm, vias 0 -> 2
- added copper zone on F.Cu, net GND
Other:
- board size 240 x 190 mm -> 320 x 280 mm
- copper layers 2 -> 4
